File: plaits/hardware_design/pcb/plaits_v50.sch (EAGLE design)
At the start: 159 parts, among them IC1 R-78E3.3-0.5, IC2 TLC59281DBQ, IC3 LD2981ABU33, IC4 STM32F373CCT6, IC5 PCM5100APW, IC6 MCP6004, IC7 MCP6004, IC8 TL072PW, IC9 LM4040B10, J1 PJ301_THONKICONN6, J10 PJ301_THONKICONN6, J2 PJ301_THONKICONN6, J3 PJ301_THONKICONN6, J4 PJ301_THONKICONN6, J5 PJ301_THONKICONN6, J6 PJ301_THONKICONN6, J7 PJ301_THONKICONN6, J8 PJ301_THONKICONN6, J9 PJ301_THONKICONN6, Q1 8MHz

Commit message: converting mini packages to 603, all done, CRC check ok.
Parts:
- C12, C17, C18, C27, C28, C33, C34, C35, C37, C40, C41, C42, C43, C44, C45, C48, C49, C50, C51, C52, C53, C6, C8: device rcl:C-USC0402 -> rcl:C-USC0603
- R10, R11, R12, R13, R15, R16, R19, R20, R21, R22, R23, R27, R28, R29, R3, R34, R35, R36, R37, R38, R39, R45, R48, R49, R50, R51, R9: device rcl:R-US_R0402 -> rcl:R-US_R0603
