File: blades/hardware_design/pcb/blades_v41/blades_v40.kicad_pcb (KiCad board)
At the start: 4 copper layers, 88.9 x 106 mm, 406 parts, among them IC1 OPA1679PW, IC10 LM4041DBZ, IC11 LM4041DBZ, IC12 SSM2164S, IC13 SSM2164S, IC14 OPA1679PW, IC15 OPA1679PW, IC16 SSM2164S, IC17 SSM2164S, IC18 OPA1679PW, IC19 TL074PW, IC2 OPA1679PW, IC20 TL074PW, IC21 OPA1679PW, IC3 TL074PW, IC4 SSM2164S, IC5 SSM2164S, IC6 OPA1678DGK, IC7 OPA1678DGK, IC8 OPA1679PW, IC9 OPA1678DGK, J1 PJ301_THONKICONNTME, J10 PJ301_THONKICONNTME, J11 PJ301_THONKICONNTME, J12 PJ301_THONKICONNTME, J13 PJ301_THONKICONNTME, J14 PJ301_THONKICONNTME, J15 PJ301_THONKICONNTME, J16 PJ301_THONKICONNTME, J2 PJ301_THONKICONNTME, J3 PJ301_THONKICONNTME, J4 PJ301_THONKICONNTME, J5 PJ301_THONKICONNTME, J6 PJ301_THONKICONNTME, J7 PJ301_THONKICONNTME, J8 PJ301_THONKICONNTME, J9 PJ301_THONKICONNTME, P1 PTCSMD, SW1 LP4ee1PBCT

Commit message: cleaned up blades dir
Other:
- board text added: "production Apr/2023 by @mb"
Changed lines of the file:
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@@
     (effects (font (size 0.8636 0.8636) (thickness 0.1524)) (justify right top mirror))
   )
-  (gr_text "cc-by-sa É. Gillet" (at 141.8336 113.8936) (layer "F.Mask")
+  (gr_text "cc-by-sa É. Gillet" (at 142.6464 55.8546) (layer "F.Mask")
     (effects (font (size 0.82042 0.82042) (thickness 0.14478)) (justify left bottom))
   )
-  (gr_text "2019. v4" (at 145.3261 115.481) (layer "F.Mask")
+  (gr_text "2019. v4" (at 145.7452 57.4294) (layer "F.Mask")
     (effects (font (size 0.8636 0.8636) (thickness 0.1524)) (justify left bottom))
   )
-  (gr_text "Blades" (at 143.2623 111.3537) (layer "F.Mask")
+  (gr_text "Blades" (at 144.2974 54.4576) (layer "F.Mask")
     (effects (font (size 1.64084 1.64084) (thickness 0.28956)) (justify left bottom))
   )
+  (gr_text "production Apr/2023 by @mb" (at 138.8364 115.1382) (layer "F.Mask")
+    (effects (font (size 0.8636 0.8636) (thickness 0.1524)) (justify left bottom))
+  )
   (segment (start 119.6432 67.4495) (end 119.6432 66.2688) (width 0.254) (layer "F.Cu") (net 1))
