File: shelves/hardware_design/pcb/shelves_v60/shelves_v60.kicad_pcb (KiCad board)
At the start: 2 copper layers, 88.9 x 107.6 mm, 248 parts, among them IC1 LM4040B10, IC10 TL074D, IC11 V2164SZ, IC12 TL072D, IC13 TL072D, IC14 TL072D, IC2 LM4040B10, IC3 TL072D, IC4 TL074D, IC5 V2164SZ, IC6 TL074D, IC7 TL074D, IC8 V2164SZ, IC9 TL074D, J1 PJ301_THONKICONN6, J10 PJ301_THONKICONN6, J11 PJ301_THONKICONN6, J12 PJ301_THONKICONN6, J13 PJ301_THONKICONN6, J14 PJ301_THONKICONN6, J15 PJ301_THONKICONN6, J16 PJ301_THONKICONN6, J17 PJ301_THONKICONN6, J18 PJ301_THONKICONN6, J19 PJ301_THONKICONN6, J2 PJ301_THONKICONN6, J20 PJ301_THONKICONN6, J3 PJ301_THONKICONN6, J4 PJ301_THONKICONN6, J5 PJ301_THONKICONN6, J6 PJ301_THONKICONN6, J7 PJ301_THONKICONN6, J8 PJ301_THONKICONN6, J9 PJ301_THONKICONN6, P1 PTCSMD, Q1 MMBT3904

Commit message: ..shelves kicad..
Parts:
- IC1, IC2: value LM4040B10 -> LM4041DBZ
- IC11, IC5, IC8: value V2164SZ -> SSM2164S
- JP5: value (none) -> M03PTH
- moved R127 1.34 mm to (184.5, 111.8)
- moved R128 1.30 mm to (184.4, 127.1)
- moved R125 1.26 mm to (184.4, 81.1)
- moved R124 1.16 mm to (184.3, 65.7)
- moved R108 1.03 mm to (169.7, 142.1)
- moved R126 0.98 mm to (184.6, 96.6)
- moved C2 0.78 mm to (178.3, 57.7)
- moved R123 0.76 mm to (181.6, 53.6)
Connections:
- net BP_1 renamed /shelves_v60_3/BP_1
- net BP_2 renamed /shelves_v60_4/BP_2
- net HP_1 renamed /shelves_v60_3/HP_1
- net HP_2 renamed /shelves_v60_4/HP_2
- net IN_INV renamed Net-(IC12A-OUT)
- net IN_INV1 renamed Net-(IC13B-OUT)
- net J_HF_CV renamed Net-(J2-3)
- net J_HF_F renamed Net-(J1-3)
- net J_IN renamed Net-(J13-3)
- net J_LF_CV renamed Net-(J10-3)
- net J_LF_F renamed Net-(J9-3)
- net LP renamed Net-(IC3A-OUT)
- net LP1 renamed Net-(IC3B-OUT)
- net MID1_F1 renamed Net-(IC8A-CTRL)
- net MID1_F2 renamed Net-(IC11A-CTRL)
- net OUTPUT renamed /shelves_v60_1/OUTPUT
- IC11 pad 1: (no net) -> unconnected-(IC11E-MODE-Pad1)
- IC5 pad 1: (no net) -> unconnected-(IC5E-MODE-Pad1)
- IC8 pad 1: (no net) -> unconnected-(IC8E-MODE-Pad1)
- J1 pad P2: (no net) -> unconnected-(J1-2-PadP2)
- J10 pad P2: (no net) -> unconnected-(J10-2-PadP2)
- J11 pad P2: (no net) -> unconnected-(J11-2-PadP2)
- J12 pad P2: (no net) -> unconnected-(J12-2-PadP2)
- J13 pad P2: (no net) -> unconnected-(J13-2-PadP2)
- J14 pad P2: (no net) -> unconnected-(J14-2-PadP2)
- J15 pad P2: (no net) -> unconnected-(J15-2-PadP2)
- J16 pad P2: (no net) -> unconnected-(J16-2-PadP2)
- J17 pad P2: (no net) -> unconnected-(J17-2-PadP2)
- J18 pad P2: (no net) -> unconnected-(J18-2-PadP2)
- J19 pad P2: (no net) -> unconnected-(J19-2-PadP2)
- J2 pad P2: (no net) -> unconnected-(J2-2-PadP2)
- J20 pad P2: (no net) -> unconnected-(J20-2-PadP2)
- J3 pad P2: (no net) -> unconnected-(J3-2-PadP2)
- J4 pad P2: (no net) -> unconnected-(J4-2-PadP2)
- J5 pad P2: (no net) -> unconnected-(J5-2-PadP2)
- J6 pad P2: (no net) -> unconnected-(J6-2-PadP2)
- J7 pad P2: (no net) -> unconnected-(J7-2-PadP2)
- J8 pad P2: (no net) -> unconnected-(J8-2-PadP2)
- J9 pad P2: (no net) -> unconnected-(J9-2-PadP2)
- JP5 pad 1: (no net) -> unconnected-(JP5-Pad1)
Routing:
- net IN: track 205.9 -> 201.4 mm
- net VCC: track 581.6 -> 580.4 mm
- net AREF_-10: track 269.4 -> 270.4 mm
- net Net-(R101-S): track 1.93 -> 2.91 mm
- net Net-(J17-3): track 3.80 -> 4.72 mm
- net Net-(J16-3): track 4.15 -> 5.02 mm
- net Net-(IC9C-OUT): track 55.7 -> 54.9 mm
- net Net-(J20-3): track 3.99 -> 4.83 mm
- net Net-(J15-3): track 5.75 -> 6.54 mm
- net Net-(J19-3): track 4.02 -> 4.80 mm
- net Net-(IC6C-OUT): track 44.1 -> 44.8 mm
- net PLUS_BUS: track 122.3 -> 123.0 mm
- net /shelves_v60_3/BP_1: track 66.9 -> 67.5 mm
- net Net-(J18-3): track 4.18 -> 4.69 mm

Commit message: preped shelves kicad
Parts:
- J1, J10, J11, J12, J13, J14, J15, J16, J17, J18, J19, J2, J20, J3, J4, J5, J6, J7, J8, J9: footprint shelves_v60:WQP_PJ_301M6 -> SynthLib:PJ_301M6
- moved R49 1.57 mm to (168.5, 94.3)
- moved R83 1.10 mm to (168.8, 117.8)
- moved U$2 0.86 mm to (167.1, 157.5)
Routing:
- net Net-(IC10A--IN): track 58.3 -> 54.8 mm
- net Net-(R36-S): track 1.93 -> 3.28 mm
- net Net-(R69-S): track 1.93 -> 2.81 mm
- net GND: vias 146 -> 145
Other:
- board text added: "cc-by-sa Émilie Gillet, 2014. v6"
- board text added: "production run @mb 7/2023"
- board text removed: "2014. v6"
- board text removed: "cc-by-sa Émilie Gillet,"
